File: Hardware/openxenium-qpi.kicad_pcb (KiCad board)
At the start: 2 copper layers, 39.4 x 36.2 mm, 36 parts, among them J1 TE Connectivity 1-2367196-0, J2 Molex 503763-0591, U1 VQFP-100_14x14mm_P0.5mm, U2 SOIC-8_5.23x5.23mm_P1.27mm, U3 SOIC-8_5.23x5.23mm_P1.27mm, U4 SOIC-8_5.23x5.23mm_P1.27mm, U5 onsemi NCV8164ASN120T1G

Commit message: HW: Import Rev. 20230304 QPI board
Parts:
- added R9: 10k, R0603, B.Cu at (134.9, 87.9)
- added TP2: TPTP13SQ, TP13SQ, F.Cu at (134.5, 87.9)
- added VCC1: SMD-Pad_0.6x1mm, SMD-Pad_0.6x1mm, F.Cu at (141.2, 95.5)
- added VCC2: SMD-Pad_0.6x1mm, SMD-Pad_0.6x1mm, F.Cu at (148.8, 95.5)
- added VCC3: SMD-Pad_0.6x1mm, SMD-Pad_0.6x1mm, F.Cu at (156.4, 95.5)
- moved J2 0.50 mm to (153.7, 117.0)
Connections:
- U1 pad 3: MOSFET_A20M -> ~{SMI}
- U1 pad 34: (no net) -> QPI_CS3
- U1 pad 4: MOSFET_D0 -> MOSFET_A20M
- U1 pad 5: ~{SMI} -> MOSFET_D0
Routing:
- net QPI_CS3: track 0.00 -> 23.6 mm, vias 0 -> 3
- net +3V3: track 18.8 -> 22.1 mm
- net ~{SMI}: track 34.8 -> 34.1 mm
Other:
- board text added: "CS0"
- board text added: "CS1"
- board text added: "CS2"
- board text added: "CS3"
- board text added: "Rev. 20230304"
- board text removed: "Rev. 20220704"
